File: analog.brd (EAGLE design)
At the start: 83.8 x 68.9 mm, 37 parts, among them Q2 IRF9530, U2 PTR08100W

Commit message: Projet Globe V0.5 Synchro added
Parts:
- removed SV5: (no value), con-lstb:MA03-1
- added U$10, U$11, U$12, U$3, U$4, U$5, U$6, U$7, U$8, U$9: JUMPER_CONNECTOR, perso:JUMPER_CONNECTOR
Connections:
- removed net M_ALIM: Q2.S, R3.1, SV5.2
- net 12V_FUSIBLE: now also Q2.S, R3.1; no longer SV5.3
- net 5V: no longer SV5.1
Routing:
- net M_ALIM: track 47.3 -> 0.00 mm
- net 12V_FUSIBLE: track 178.4 -> 221.5 mm
- net 5V: track 223.7 -> 220.7 mm
Changed lines of the file:
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@@
 <attribute name="OC_FARNELL" value="unknown" x="52.07" y="6.35" size="1.778" layer="27" rot="R90" display="off"/>
-</element>
-<element name="SV5" library="con-lstb" package="MA03-1" value="" x="35.56" y="57.15" rot="R90">
-<attribute name="OC_NEWARK" value="unknown" x="35.56" y="57.15" size="1.778" layer="27" rot="R90" display="off"/>
-<attribute name="MPN" value="" x="35.56" y="57.15" size="1.778" layer="27" rot="R90" display="off"/>
-<attribute name="MF" value="" x="35.56" y="57.15" size="1.778" layer="27" rot="R90" display="off"/>
-<attribute name="OC_FARNELL" value="unknown" x="35.56" y="57.15" size="1.778" layer="27" rot="R90" display="off"/>
 </element>
 <element name="SV6" library="con-lstb" package="MA04-1" value="" x="55.88" y="43.18" rot="R90">
@@
 <attribute name="OC_FARNELL" value="unknown" x="62.23" y="13.97" size="1.778" layer="27" display="off"/>
 </element>
+<element name="U$3" library="perso" package="JUMPER_CONNECTOR" value="JUMPER_CONNECTOR" x="5.715" y="0.635"/>
+<element name="U$4" library="perso" package="JUMPER_CONNECTOR" value="JUMPER_CONNECTOR" x="5.715" y="10.16"/>
+<element name="U$5" library="perso" package="JUMPER_CONNECTOR" value="JUMPER_CONNECTOR" x="15.24" y="0.635"/>
+<element name="U$6" library="perso" package="JUMPER_CONNECTOR" value="JUMPER_CONNECTOR" x="83.185" y="64.135"/>
+<element name="U$7" library="perso" package="JUMPER_CONNECTOR" value="JUMPER_CONNECTOR" x="96.52" y="53.34"/>
+<element name="U$8" library="perso" package="JUMPER_CONNECTOR" value="JUMPER_CONNECTOR" x="31.115" y="-6.35"/>
+<element name="U$9" library="perso" package="JUMPER_CONNECTOR" value="JUMPER_CONNECTOR" x="25.4" y="-6.35"/>
+<element name="U$10" library="perso" package="JUMPER_CONNECTOR" value="JUMPER_CONNECTOR" x="94.615" y="59.69"/>
+<element name="U$11" library="perso" package="JUMPER_CONNECTOR" value="JUMPER_CONNECTOR" x="17.145" y="-6.985"/>
+<element name="U$12" library="perso" package="JUMPER_CONNECTOR" value="JUMPER_CONNECTOR" x="90.805" y="64.135"/>
 </elements>
 <signals>
@@
 <contactref element="C2" pad="+"/>
 <contactref element="SV4" pad="3"/>
-<contactref element="SV5" pad="1"/>
 <contactref element="SV6" pad="4"/>
 <contactref element="F1" pad="2"/>
@@
 <wire x1="67.31" y1="13.97" x2="67.31" y2="3.81" width="1.9304" layer="1"/>
 <wire x1="67.31" y1="3.81" x2="64.77" y2="1.27" width="1.9304" layer="1"/>
-<wire x1="35.56" y1="54.61" x2="35.56" y2="53.975" width="1.9304" layer="16"/>
-<wire x1="35.56" y1="53.975" x2="29.21" y2="47.625" width="1.9304" layer="16"/>
 <wire x1="29.21" y1="47.625" x2="29.21" y2="35.56" width="1.9304" layer="16"/>
 <wire x1="29.21" y1="35.56" x2="30.48" y2="34.29" width="1.9304" layer="16"/>
@@
 <wire x1="40.005" y1="29.21" x2="41.275" y2="27.94" width="1.9304" layer="16"/>
 <wire x1="55.245" y1="47.625" x2="55.88" y2="46.99" width="1.9304" layer="16"/>
-<wire x1="55.245" y1="47.625" x2="48.895" y2="47.625" width="1.9304" layer="16"/>
-<wire x1="48.895" y1="47.625" x2="43.18" y2="53.34" width="1.9304" layer="16"/>
-<wire x1="43.18" y1="53.34" x2="36.83" y2="53.34" width="1.9304" layer="16"/>
-<wire x1="36.83" y1="53.34" x2="35.56" y2="54.61" width="1.9304" layer="16"/>
+<wire x1="55.245" y1="47.625" x2="49.53" y2="47.625" width="1.9304" layer="16"/>
+<wire x1="49.53" y1="47.625" x2="48.895" y2="47.625" width="1.9304" layer="16"/>
 <wire x1="59.69" y1="46.99" x2="62.865" y2="50.165" width="1.9304" layer="16"/>
 <wire x1="62.865" y1="50.165" x2="62.865" y2="53.34" width="1.9304" layer="16"/>
@@
 <wire x1="46.355" y1="10.16" x2="38.735" y2="10.16" width="1.9304" layer="1"/>
 <wire x1="38.735" y1="10.16" x2="36.83" y2="12.065" width="1.9304" layer="1"/>
+<wire x1="29.21" y1="47.625" x2="31.115" y2="49.53" width="1.9304" layer="16"/>
+<wire x1="31.115" y1="49.53" x2="37.465" y2="49.53" width="1.9304" layer="16"/>
+<wire x1="37.465" y1="49.53" x2="39.37" y2="51.435" width="1.9304" layer="16"/>
+<wire x1="39.37" y1="51.435" x2="44.45" y2="51.435" width="1.9304" layer="16"/>
+<wire x1="44.45" y1="51.435" x2="48.26" y2="47.625" width="1.9304" layer="16"/>
+<wire x1="48.26" y1="47.625" x2="48.895" y2="47.625" width="1.9304" layer="16"/>
 </signal>
 <signal name="12V_FUSIBLE">
@@
 <contactref element="R12" pad="1"/>
 <contactref element="SV4" pad="1"/>
-<contactref element="SV5" pad="3"/>
 <contactref element="SV6" pad="1"/>
 <contactref element="F3" pad="2"/>
@@
 <wire x1="55.88" y1="39.37" x2="65.405" y2="39.37" width="1.9304" layer="16"/>
 <wire x1="65.405" y1="39.37" x2="67.945" y2="36.83" width="1.9304" layer="16"/>
-<wire x1="35.56" y1="59.69" x2="35.56" y2="61.595" width="1.9304" layer="16"/>
 <wire x1="83.82" y1="5.715" x2="83.82" y2="33.655" width="1.9304" layer="16"/>
 <wire x1="83.82" y1="33.655" x2="81.28" y2="36.195" width="1.9304" layer="16"/>
@@
 <wire x1="80.01" y1="37.465" x2="68.58" y2="37.465" width="1.9304" layer="16"/>
 <wire x1="68.58" y1="37.465" x2="67.945" y2="36.83" width="1.9304" layer="16"/>
-<wire x1="35.56" y1="61.595" x2="38.1" y2="64.135" width="1.9304" layer="16"/>
-<wire x1="38.1" y1="64.135" x2="78.74" y2="64.135" width="1.9304" layer="16"/>
+<wire x1="30.48" y1="64.135" x2="78.74" y2="64.135" width="1.9304" layer="16"/>
 <wire x1="83.82" y1="59.055" x2="78.74" y2="64.135" width="1.9304" layer="16"/>
+<contactref element="Q2" pad="S"/>
+<wire x1="25.4" y1="53.34" x2="26.67" y2="54.61" width="1.9304" layer="16"/>
+<wire x1="15.24" y1="63.5" x2="23.495" y2="63.5" width="1.9304" layer="16"/>
+<wire x1="11.43" y1="56.515" x2="18.415" y2="56.515" width="1.9304" layer="16"/>
+<wire x1="18.415" y1="56.515" x2="21.59" y2="53.34" width="1.9304" layer="16"/>
+<wire x1="21.59" y1="53.34" x2="25.4" y2="53.34" width="1.9304" layer="16"/>
+<contactref element="R3" pad="1"/>
+<wire x1="26.67" y1="54.61" x2="26.67" y2="60.325" width="1.9304" layer="16"/>
+<wire x1="26.67" y1="60.325" x2="23.495" y2="63.5" width="1.9304" layer="16"/>
+<wire x1="30.48" y1="64.135" x2="26.67" y2="60.325" width="1.9304" layer="16"/>
+<wire x1="15.24" y1="63.5" x2="15.875" y2="63.5" width="0" layer="19" extent="16-16"/>
 </signal>
 <signal name="VO_ADJ">
@@
 <wire x1="58.4454" y1="7.6454" x2="60.96" y2="10.16" width="1.9304" layer="16"/>
 </signal>
-<signal name="M_ALIM">
-<contactref element="Q2" pad="S"/>
-<contactref element="SV5" pad="2"/>
-<wire x1="25.4" y1="53.34" x2="26.67" y2="54.61" width="1.9304" layer="16"/>
-<wire x1="26.67" y1="54.61" x2="26.67" y2="59.69" width="1.9304" layer="16"/>
-<wire x1="26.67" y1="59.69" x2="27.94" y2="60.96" width="1.9304" layer="16"/>
-<wire x1="27.94" y1="60.96" x2="31.115" y2="60.96" width="1.9304" layer="16"/>
-<contactref element="R3" pad="1"/>
-<wire x1="31.115" y1="60.96" x2="32.385" y2="59.69" width="1.9304" layer="16"/>
-<wire x1="32.385" y1="59.69" x2="32.385" y2="57.785" width="1.9304" layer="16"/>
-<wire x1="32.385" y1="57.785" x2="33.02" y2="57.15" width="1.9304" layer="16"/>
-<wire x1="33.02" y1="57.15" x2="35.56" y2="57.15" width="1.9304" layer="16"/>
-<wire x1="15.24" y1="63.5" x2="22.86" y2="63.5" width="1.9304" layer="16"/>
-<wire x1="22.86" y1="63.5" x2="26.67" y2="59.69" width="1.9304" layer="16"/>
-<wire x1="11.43" y1="56.515" x2="18.415" y2="56.515" width="1.9304" layer="16"/>
-<wire x1="18.415" y1="56.515" x2="21.59" y2="53.34" width="1.9304" layer="16"/>
-<wire x1="21.59" y1="53.34" x2="25.4" y2="53.34" width="1.9304" layer="16"/>
-<wire x1="15.24" y1="63.5" x2="15.875" y2="63.5" width="0" layer="19" extent="16-16"/>
-</signal>
 <signal name="R_STRIP_5">
